File: Brooder_sch_v1.2.1.brd (EAGLE design)
At the start: 100 x 90 mm, 38 parts, among them J1 DCJ0202, J2 1X2-3.5MM, J3 DCJ0202, J4 1X2-3.5MM, T1 2N2222, U1 328P

Commit message: Adds new file due to file locking
Parts:
- removed U$3: RTC-DS3231-AT24C32, diy-modules-1.8.0:RTC-DS3231-AT24C32
Connections:
- removed net GND.1: U$3.J1.6
- removed net GND.2: U$3.J2.4
- removed net SCL: U1.28
- removed net SDA: U1.27
- removed net VCC.1: U$3.J1.5
- removed net VCC.2: U$3.J2.3
- net PC4: now also U1.27
- net PC5: now also U1.28
Routing:
- net SCL: track 10.8 -> 0.00 mm
- net PC5: track 0.00 -> 10.8 mm
Changed lines of the file:
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@@
 <attribute name="SF_SKU" value="PRT-08432" x="49.01" y="85.56" size="1.778" layer="27" display="off"/>
 </element>
-<element name="U$3" library="diy-modules-1.8.0" package="RTC-DS3231-AT24C32" value="RTC-DS3231-AT24C32" x="20.12" y="-103.5"/>
 </elements>
 <signals>
@@
 <signal name="PC4">
 <contactref element="DS3231" pad="4"/>
+<contactref element="U1" pad="27"/>
+<wire x1="41.94" y1="53.99" x2="71.66" y2="56.3" width="0" layer="19" extent="1-1"/>
 </signal>
 <signal name="PC5">
 <contactref element="DS3231" pad="3"/>
+<contactref element="U1" pad="28"/>
+<wire x1="41.94" y1="56.53" x2="52.71" y2="56.53" width="1.27" layer="16"/>
+<wire x1="52.71" y1="56.53" x2="71.66" y2="53.76" width="0" layer="19" extent="16-16"/>
 </signal>
 <signal name="TX">
@@
 <wire x1="49.01" y1="85.56" x2="65.25" y2="85.56" width="0" layer="19" extent="1-1"/>
 </signal>
-<signal name="VCC.1">
-<contactref element="U$3" pad="J1.5"/>
-</signal>
-<signal name="GND.2">
-<contactref element="U$3" pad="J2.4"/>
-</signal>
-<signal name="VCC.2">
-<contactref element="U$3" pad="J2.3"/>
-</signal>
-<signal name="GND.1">
-<contactref element="U$3" pad="J1.6"/>
-</signal>
-<signal name="SCL">
-<contactref element="U1" pad="28"/>
-<wire x1="41.94" y1="56.53" x2="52.71" y2="56.53" width="1.27" layer="16"/>
-</signal>
-<signal name="SDA">
-<contactref element="U1" pad="27"/>
-</signal>
 </signals>
