File: Brooder_sch_v1.2.1.sch (EAGLE design)
At the start: 38 parts, among them J1 DCJ0202, J2 1X2-3.5MM, J3 DCJ0202, J4 1X2-3.5MM, T1 2N2222, U1 328P

Commit message: Adds new file due to file locking
Parts:
- removed U$3: RTC-DS3231-AT24C32, diy-modules-1.8.0:RTC-DS3231-AT24C32
Connections:
- removed net SCL: U1.PC5(ADC5/SCL)
- removed net SDA: U1.PC4(ADC4/SDA)
- net PC4: now also U1.PC4(ADC4/SDA)
- net PC5: now also U1.PC5(ADC5/SCL)
Changed lines of the file:
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@@
 <part name="GND22" library="supply1" library_urn="urn:adsk.eagle:library:371" deviceset="GND" device=""/>
 <part name="LOAD" library="SparkFun-Connectors" deviceset="CONN_02" device="5MM"/>
-<part name="U$3" library="diy-modules-1.8.0" deviceset="RTC-DS3231-AT24C32" device=""/>
 </parts>
 <sheets>
@@
 <attribute name="NAME" x="10.16" y="-20.828" size="1.778" layer="95" font="vector" rot="R180"/>
 </instance>
-<instance part="U$3" gate="G$1" x="83.82" y="-45.72"/>
 </instances>
 <busses>
@@
 <label x="101.6" y="68.58" size="1.778" layer="95"/>
 </segment>
+<segment>
+<pinref part="U1" gate="U1" pin="PC4(ADC4/SDA)"/>
+<wire x1="76.2" y1="93.98" x2="83.82" y2="93.98" width="0.1524" layer="91"/>
+<label x="83.82" y="93.98" size="1.778" layer="95"/>
+</segment>
 </net>
 <net name="PC5" class="0">
@@
 <wire x1="109.22" y1="71.12" x2="101.6" y2="71.12" width="0.1524" layer="91"/>
 <label x="101.6" y="71.12" size="1.778" layer="95"/>
+</segment>
+<segment>
+<pinref part="U1" gate="U1" pin="PC5(ADC5/SCL)"/>
+<wire x1="76.2" y1="91.44" x2="83.82" y2="91.44" width="0.1524" layer="91"/>
+<label x="83.82" y="91.44" size="1.778" layer="95"/>
 </segment>
 </net>
@@
 </segment>
 </net>
-<net name="SCL" class="0">
-<segment>
-<pinref part="U1" gate="U1" pin="PC5(ADC5/SCL)"/>
-<wire x1="76.2" y1="91.44" x2="83.82" y2="91.44" width="0.1524" layer="91"/>
-<label x="83.82" y="91.44" size="1.778" layer="95"/>
-</segment>
-</net>
-<net name="SDA" class="0">
-<segment>
-<pinref part="U1" gate="U1" pin="PC4(ADC4/SDA)"/>
-<wire x1="76.2" y1="93.98" x2="83.82" y2="93.98" width="0.1524" layer="91"/>
-<label x="83.82" y="93.98" size="1.778" layer="95"/>
-</segment>
-</net>
